Commit message: Lidar position fixed

File: f1tenth_sim/launch/ego_racecar.xacro (robot description, xacro)
@@ -8,5 +8,5 @@
   <xacro:property name="wheel_radius" value="0.0508" />
   <xacro:property name="wheel_length" value="0.0381" />
-  <xacro:property name="laser_distance_from_base_link" value="0.275" />
+  <xacro:property name="laser_distance_from_base_link" value="0.265" />
   <xacro:property name="laser_height" value="0.05" />
   <xacro:property name="laser_radius" value="0.026" />

File: f1tenth_sim/launch/opp_racecar.xacro (robot description, xacro)
@@ -8,5 +8,5 @@
   <xacro:property name="wheel_radius" value="0.0508" />
   <xacro:property name="wheel_length" value="0.0381" />
-  <xacro:property name="laser_distance_from_base_link" value="0.275" />
+  <xacro:property name="laser_distance_from_base_link" value="0.265" />
   <xacro:property name="laser_height" value="0.05" />
   <xacro:property name="laser_radius" value="0.026" />
